File: power_meter_v2.kicad_sch (KiCad schematic)
At the start: 69 parts

Commit message: Assign footprints to symbols
Parts:
- removed D?: LED_RGBA, symbol guille_3rdparty:LED_RGBA
- added D3: LED_RGBA, guille_3rdparty:APHF1608LSEEQBDZGKC, symbol guille_library:LED_RGBA
- added J1: Conn_01x04_Male, guille_3rdparty:TerminalBlock_Altech_AK300-4_P5.00mm, symbol Connector:Conn_01x04_Male
- C1, C2: renamed from C?; footprint (none) -> Capacitor_SMD:C_1206_3216Metric
- C10, C7, C8, C9: renamed from C?; footprint (none) -> Capacitor_SMD:C_0402_1005Metric
- C3, C5: renamed from C?; value C -> 100n; footprint (none) -> Capacitor_SMD:C_0402_1005Metric
- C4, C6: renamed from C?; value C -> 1u; footprint (none) -> Capacitor_SMD:C_0402_1005Metric
- D1, D2: renamed from D?; footprint (none) -> LED_SMD:LED_0402_1005Metric
- F1: renamed from F?; footprint (none) -> guille_3rdparty:Fuse_2512_6332Metric
- J2: renamed from J?; footprint (none) -> Connector_PinHeader_2.54mm:PinHeader_1x02_P2.54mm_Vertical
- J3, J4: renamed from J?; footprint (none) -> Connector_PinSocket_2.54mm:PinSocket_1x04_P2.54mm_Vertical
- R1, R2, R3: renamed from R?; footprint (none) -> Resistor_THT:R_Axial_DIN0207_L6.3mm_D2.5mm_P7.62mm_Horizontal
- R10, R11, R12, R13, R14, R15, R16, R17, R18, R19, R20, R21, R22, R23, R24, R25, R26, R27, R28, R4, R5, R6, R7, R8, R9: renamed from R?; footprint (none) -> Resistor_SMD:R_0402_1005Metric
- RV1: renamed from RV?; footprint (none) -> Varistor:RV_Disc_D12mm_W3.9mm_P7.5mm
- RV2: renamed from RV?; footprint (none) -> Potentiometer_THT:Potentiometer_Bourns_3296W_Vertical
- SW1: renamed from SW?; footprint (none) -> Button_Switch_SMD:SW_Push_1P1T_NO_6x6mm_H9.5mm
- TP1: renamed from TP?; footprint (none) -> TestPoint:TestPoint_Pad_D1.5mm
- U1, U7: renamed from U?; footprint (none) -> Package_SO:TSSOP-14_4.4x5mm_P0.65mm
- U10, U8, U9: renamed from U?; footprint (none) -> guille_library:JACK_PCB_3.5
- U11: renamed from U?; footprint (none) -> guille_3rdparty:SHT40
- U12: renamed from U?; footprint (none) -> guille_library:MS88SF3
- U3, U4, U5: renamed from U?; footprint (none) -> guille_library:ZMPT107-1
- U6: renamed from U?; footprint (none) -> guille_library:HLK-2M05
- gave numbers to parts that had none: 1
Connections:
- net LED_EXT1 is gone; now on net LED1: R13.2
- net LED_EXT2 is gone; now on net LED2: R20.2
- net +3V3: now also U12.31 (VDD), D3.1 (A); no longer U12.33 (DCCH)
- net EXT1: now also U12.20 (P0.06)
- net EXT2: now also U12.19 (P0.07)
- net I2C_SCL: now also U12.30 (P0.14)
- net I2C_SDA: now also U12.29 (P0.16)
- net L1: now also J1.2 (Pin_2)
- net L2: now also J1.3 (Pin_3)
- net L3: now also J1.4 (Pin_4)
- net LEDB: now also U12.38 (P0.19)
- net LEDG: now also U12.39 (P0.13)
- net LEDR: now also U12.40 (P0.15)
- net N: now also J1.1 (Pin_1)
- net at R21.1: now also D3.2 (RK)
- net at R26.1: now also D3.4 (BK)
- net at R25.1: now also D3.3 (GK)
- net LED2: now reaches U12.41 (P0.17)
- net LED1: now reaches U12.42 (P0.21)
- no-connect marks 3 -> 36
Other:
- note added: "TODO: Add analog filters"
- note removed: "TODO: Check LEDs colors!!!"
- moved on the sheet: C7, D1, D2, R13, R20, R21, R25, R26, U11

Commit message: New sheet for pwr measure sch and add lps25 symbol
Parts:
- removed C3, C5: 100n, Capacitor_SMD:C_0402_1005Metric, symbol Device:C
- removed C4, C6: 1u, Capacitor_SMD:C_0402_1005Metric, symbol Device:C
- removed J1: Conn_01x04_Male, guille_3rdparty:TerminalBlock_Altech_AK300-4_P5.00mm, symbol Connector:Conn_01x04_Male
- removed R1, R2, R3: 820k, Resistor_THT:R_Axial_DIN0207_L6.3mm_D2.5mm_P7.62mm_Horizontal, symbol Device:R
- removed R10, R11, R12: 200k, Resistor_SMD:R_0402_1005Metric, symbol Device:R
- removed R14, R15, R16, R4, R5, R6: 100, Resistor_SMD:R_0402_1005Metric, symbol Device:R
- removed R17, R18, R19, R7, R8, R9: 10k, Resistor_SMD:R_0402_1005Metric, symbol Device:R
- removed R22, R23, R24: 3k9, Resistor_SMD:R_0402_1005Metric, symbol Device:R
- removed RV2: Trim, Potentiometer_THT:Potentiometer_Bourns_3296W_Vertical, symbol Device:R_Potentiometer_Trim
- removed TP1: TestPoint, TestPoint:TestPoint_Pad_D1.5mm, symbol Connector:TestPoint
- removed U1, U7: MCP6004, Package_SO:TSSOP-14_4.4x5mm_P0.65mm, symbol Amplifier_Operational:MCP6004
- removed U10, U8, U9: JACK_PCB_3.5, guille_library:JACK_PCB_3.5, symbol guille_library:JACK_PCB_3.5
- removed U3, U4, U5: ZMPT107-1, guille_library:ZMPT107-1, symbol guille_library:ZMPT107-1
- added C?: 100n, Capacitor_SMD:C_0402_1005Metric, symbol Device:C
- added H1, H2, H3, H4: MountingHole, MountingHole:MountingHole_3.2mm_M3_ISO7380, symbol Mechanical:MountingHole
- added J?: Screw_Terminal_01x04, symbol Connector:Screw_Terminal_01x04
- added U?: LPS25HB, Package_LGA:ST_HLGA-10_2.5x2.5mm_P0.6mm_LayoutBorder3x2y, symbol Sensor_Pressure:LPS25HB
- renumbered C7 to C3, C8 to C4, C9 to C5, C10 to C6, R13 to R1, R20 to R2, R21 to R3, R25 to R4, R26 to R5, R27 to R6, R28 to R7, U2 to U1, U6 to U2, U11 to U3, U12 to U4
Connections:
- net +3V3: now also C?.1, U?.1 (VDDio), U?.10 (VDD), U?.6 (~{CS})
- net GND: now also C?.2, U?.3 (GND), U?.8 (GND), U?.9 (GND)
- net I2C_SCL: now also U?.2 (SCL/SCLK)
- net I2C_SDA: now also U?.4 (SDA/MOSI)
- net L1: now also J?.2 (Pin_2)
- net L2: now also J?.3 (Pin_3)
- net L3: now also J?.4 (Pin_4)
- net N: now also J?.1 (Pin_1)
- net LPS_INT: now reaches U4.52 (P1.02)
- net LPS_INT: now also U?.7 (INT_DRDY)
- no-connect marks 36 -> 33
Other:
- added sheet power_measurement (power_measurement.kicad_sch)
- note removed: "TODO: Connect GPIOs and set unconnected pins"
